File: KC_NixieBargraphHat/NixieBargraphHat.sch (KiCad schematic (older format))
At the start: 49 parts, among them J1 Screw_Terminal_1x03, J2 Screw_Terminal_1x02, J3 Screw_Terminal_1x03, J4 Screw_Terminal_1x03, Q1 FDD18N20LZ, Q2 2N7002, Q3 FDD18N20LZ, Q4 2N7002, U1 MCP6411, U2 Raspberry_PI_Zero_Header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

Commit message: updated the schematic with dual solution for left and right channels
Parts:
- added C?: 1uF, symbol C
Connections:
- net +3V3: now also C?.1
- net GND: now also C?.2
Changed lines of the file:
@@
 $EndComp
 Wire Wire Line
-	5650 2650 5650 3050
-Wire Wire Line
-	5650 3050 5650 3200
+	5650 2650 5650 3200
 Wire Wire Line
 	5650 3500 5650 3600
 Wire Wire Line
-	4350 2650 4450 2650
-Wire Wire Line
-	4450 2650 4800 2650
-Wire Wire Line
-	2350 2100 2500 2100
-Wire Wire Line
-	2500 2100 3250 2100
-Wire Wire Line
-	3250 2100 3600 2100
+	4350 2650 4800 2650
+Wire Wire Line
+	2350 2100 3600 2100
 Wire Wire Line
 	3600 2100 3600 2550
@@
 	3600 2550 3750 2550
 Wire Wire Line
-	3600 2750 3700 2750
-Wire Wire Line
-	3700 2750 3750 2750
+	3600 2750 3750 2750
 Connection ~ 5650 3050
 Wire Wire Line
@@
 	5650 950  5650 1050
 Wire Wire Line
-	5650 2100 5650 2150
-Wire Wire Line
-	5650 2150 5650 2250
-Wire Wire Line
-	5650 1350 5650 1450
-Wire Wire Line
-	5650 1450 5650 1500
+	5650 2100 5650 2250
+Wire Wire Line
+	5650 1350 5650 1500
 Wire Wire Line
 	2500 2200 2500 2100
 Connection ~ 2500 2100
 Wire Wire Line
-	2950 1300 2950 1800
-Wire Wire Line
-	2950 1800 2950 2400
+	2950 1300 2950 2400
 Wire Wire Line
 	3150 2700 3250 2700
@@
 	2950 3100 2950 3000
 Wire Wire Line
-	3950 1300 3950 1900
-Wire Wire Line
-	3950 1900 3950 2350
+	3950 1300 3950 2350
 Wire Wire Line
 	5200 2650 5100 2650
@@
 	8850 2150 9400 2150
 Wire Wire Line
-	9400 2000 9400 2150
-Wire Wire Line
-	9400 2150 9400 2350
+	9400 2000 9400 2350
 Wire Wire Line
 	9400 2350 8850 2350
@@
 	9550 4350 9550 4250
 Wire Wire Line
-	9550 4250 9650 4250
-Wire Wire Line
-	9650 4250 9900 4250
+	9550 4250 9900 4250
 Text Notes 9900 4600 0    60   ~ 0
 R-Pi Zero GPIO #18 (BCD)
@@
 	9100 4850 9250 4850
 Wire Wire Line
-	9250 4550 9250 4850
-Wire Wire Line
-	9250 4850 9250 5350
-Wire Wire Line
-	9250 5350 9250 6000
+	9250 4550 9250 6000
 Wire Wire Line
 	9100 5350 9250 5350
@@
 	8400 5850 8600 5850
 Wire Wire Line
-	8400 4350 8400 5150
-Wire Wire Line
-	8400 5150 8400 5850
-Wire Wire Line
-	8400 5850 8400 6000
+	8400 4350 8400 6000
 Wire Wire Line
 	8600 5150 8400 5150
@@
 	9450 4050 9100 4050
 Wire Wire Line
-	9450 3500 9450 3950
-Wire Wire Line
-	9450 3950 9450 4050
+	9450 3500 9450 4050
 Wire Wire Line
 	9100 3950 9450 3950
@@
 	8600 3950 8350 3950
 Wire Wire Line
-	8350 3500 8350 3950
-Wire Wire Line
-	8350 3950 8350 4750
+	8350 3500 8350 4750
 Wire Wire Line
 	8350 4750 8600 4750
@@
 PWM_0_50Hz
 Wire Wire Line
-	3950 1900 4300 1900
-Wire Wire Line
-	4300 1900 4600 1900
+	3950 1900 4600 1900
 $Comp
 L +5V #PWR9
@@
 $EndComp
 Wire Wire Line
-	6000 6000 6000 6400
-Wire Wire Line
-	6000 6400 6000 6550
+	6000 6000 6000 6550
 Wire Wire Line
 	6000 6850 6000 6950
 Wire Wire Line
-	4700 6000 4800 6000
-Wire Wire Line
-	4800 6000 5150 6000
-Wire Wire Line
-	2700 5450 2850 5450
-Wire Wire Line
-	2850 5450 3600 5450
-Wire Wire Line
-	3600 5450 3950 5450
+	4700 6000 5150 6000
+Wire Wire Line
+	2700 5450 3950 5450
 Wire Wire Line
 	3950 5450 3950 5900
@@
 	3950 5900 4100 5900
 Wire Wire Line
-	4100 6100 4050 6100
-Wire Wire Line
-	4050 6100 3950 6100
+	3950 6100 4100 6100
 Wire Wire Line
 	4050 6100 4050 6400
@@
 	6000 4300 6000 4400
 Wire Wire Line
-	6000 5450 6000 5500
-Wire Wire Line
-	6000 5500 6000 5600
-Wire Wire Line
-	6000 4700 6000 4800
-Wire Wire Line
-	6000 4800 6000 4850
+	6000 5450 6000 5600
+Wire Wire Line
+	6000 4700 6000 4850
 Wire Wire Line
 	2850 5550 2850 5450
 Connection ~ 2850 5450
 Wire Wire Line
-	3300 4650 3300 5250
-Wire Wire Line
-	3300 5250 3300 5750
+	3300 4650 3300 5750
 Wire Wire Line
 	3500 6050 3600 6050
@@
 	3300 6450 3300 6350
 Wire Wire Line
-	4300 4650 4300 5250
-Wire Wire Line
-	4300 5250 4300 5700
+	4300 4650 4300 5700
 Wire Wire Line
 	5550 6000 5450 6000
@@
 R-Pi Zero GPIO #6 (BCD)
 Wire Wire Line
-	4300 5250 4650 5250
-Wire Wire Line
-	4650 5250 4950 5250
+	4300 5250 4950 5250
 $Comp
 L +5V #PWR12
@@
 Connection ~ 4300 5250
 Wire Wire Line
-	9750 3900 9750 4150
-Wire Wire Line
-	9750 4150 9750 4650
+	9750 3900 9750 4650
 Wire Wire Line
 	9750 3900 9900 3900
@@
 PWM_1_50Hz
 Wire Wire Line
-	7900 5250 7900 5350
-Wire Wire Line
-	7900 5350 7900 5450
+	7900 5250 7900 5450
 Wire Wire Line
 	7900 5250 7750 5250
@@
 	5450 6400 6000 6400
 Wire Wire Line
-	4050 6400 4800 6400
-Wire Wire Line
-	4800 6400 5150 6400
+	4050 6400 5150 6400
 $Comp
 L R R8
@@
 Connection ~ 3700 2750
 Wire Wire Line
-	3700 3050 4450 3050
-Wire Wire Line
-	4450 3050 4800 3050
+	3700 3050 4800 3050
 $Comp
 L D_x2_Serial_AKC D4
@@
 $EndComp
 Wire Wire Line
-	7750 5550 7900 5550
-Wire Wire Line
-	7900 5550 8050 5550
+	7750 5550 8050 5550
 Wire Wire Line
 	8350 5550 8600 5550
@@
 $EndComp
 Wire Wire Line
-	9550 4450 9850 4450
-Wire Wire Line
-	9850 4450 10050 4450
+	9550 4450 10050 4450
 $Comp
 L R R24
@@
 	4800 6350 4800 6400
 Connection ~ 4800 6400
+$Comp
+L C C?
+U 1 1 5C3FF84B
+P 3250 1500
+F 0 "C?" H 3275 1600 50  0000 L CNN
+F 1 "1uF" H 3275 1400 50  0000 L CNN
+F 2 "" H 3288 1350 50  0001 C CNN
+F 3 "" H 3250 1500 50  0001 C CNN
+	1    3250 1500
+	1    0    0    -1
+$EndComp
+$Comp
+L GND #PWR?
+U 1 1 5C3FF921
+P 3250 1650
+F 0 "#PWR?" H 3250 1400 50  0001 C CNN
+F 1 "GND" H 3250 1500 50  0000 C CNN
+F 2 "" H 3250 1650 50  0001 C CNN
+F 3 "" H 3250 1650 50  0001 C CNN
+	1    3250 1650
+	1    0    0    -1
+$EndComp
+Wire Wire Line
+	3250 1350 2950 1350
+Connection ~ 2950 1350
 $EndSCHEMATC

Commit message: updated layout files.
Parts:
- C1, C5: footprint (none) -> Capacitors_SMD:C_0805_HandSoldering; MPN (none) -> C0805C332KDRACAUTO
- C2, C6: footprint (none) -> Capacitors_SMD:C_0805_HandSoldering; MPN (none) -> C0805C104K3RACTU
- C3, C7: footprint (none) -> Capacitors_SMD:C_0805_HandSoldering; MPN (none) -> CL21F105ZBFNNNE
- C4: renamed from C?; footprint (none) -> Capacitors_SMD:C_0805_HandSoldering; MPN (none) -> CL21F105ZBFNNNE
- C8, C9: renamed from C?; value 0.1uF -> 1nF; footprint (none) -> Capacitors_SMD:C_0805_HandSoldering; MPN (none) -> C0805C102J5HACAUTO
- D1, D2, D3, D4: value D_x2_Serial_AKC -> BAV99; footprint (none) -> TO_SOT_Packages_SMD:SOT-23; MPN (none) -> BAV99,235
- J1, J3, J4: footprint (none) -> TerminalBlock_Phoenix:TerminalBlock_Phoenix_MPT-2.54mm_3pol; MPN (none) -> 1725669
- J2: footprint (none) -> TerminalBlock_Phoenix:TerminalBlock_Phoenix_MPT-2.54mm_2pol; MPN (none) -> 1725656
- N1, N2: footprint nixies-us_IN-9 -> (none)
- Q1, Q3: footprint TO_SOT_Packages_SMD:SOT-223-3Lead_TabPin2 -> TO_SOT_Packages_SMD:TO-252-2Lead; MPN (none) -> FDD18N20LZ
- Q2, Q4: MPN (none) -> 2N7002-TP
- R1, R10, R5, R6, R7, R8: footprint (none) -> Resistors_SMD:R_0805_HandSoldering; MPN (none) -> RC0805FR-071KL
- R11, R3: value 3.3k 2W -> 1k 2W; footprint (none) -> Resistors_THT:R_Axial_DIN0411_L9.9mm_D3.6mm_P12.70mm_Horizontal; MPN (none) -> PR02000201001JR500
- R12, R4: footprint (none) -> Resistors_SMD:R_0805_HandSoldering; MPN (none) -> RC0805FR-07133RL
- R13, R14: footprint (none) -> Resistors_SMD:R_0805_HandSoldering; MPN (none) -> CRGCQ0805F220K
- R15, R16, R17, R18, R19, R20, R21, R22, R23, R24: footprint (none) -> Resistors_SMD:R_0805_HandSoldering
- R2, R9: value 15k -> 8.2k; footprint (none) -> Resistors_SMD:R_0805_HandSoldering; MPN (none) -> RC0805FR-078K2L
- U1, U3: footprint (none) -> TO_SOT_Packages_SMD:SOT-23-5_HandSoldering; MPN (none) -> MCP6411T-E/OT
- U2: footprint (none) -> etaclock:Raspberry_Pi_Zero_40pins
Connections:
- net +5V: now also J1.1; no longer J1.3
- net GND: now also J1.3, U2.41 (MountHoles); no longer J1.1
Other:
- moved on the sheet: R18

Commit message: Updated the BOM to a different FET that is in stock  250v
Parts:
- Q1, Q3: value FDD18N20LZ -> FDD7N25LZTM; MPN FDD18N20LZ -> FDD7N25LZTM
Changed lines of the file:
@@
 P 5550 2450
 F 0 "Q1" H 5750 2525 50  0000 L CNN
-F 1 "FDD18N20LZ" H 5750 2450 50  0000 L CNN
+F 1 "FDD7N25LZTM" H 5750 2450 50  0000 L CNN
 F 2 "TO_SOT_Packages_SMD:TO-252-2Lead" H 5750 2375 50  0001 L CIN
-F 3 "https://www.digikey.com/product-detail/en/on-semiconductor/FDD18N20LZ/FDD18N20LZCT-ND/3908087" H 5550 2450 50  0001 L CNN
-F 4 "FDD18N20LZ" H 5550 2450 60  0001 C CNN "MPN"
+F 3 "https://www.digikey.com/product-detail/en/on-semiconductor/FDD7N25LZTM/FDD7N25LZTMCT-ND/3908038" H 5550 2450 50  0001 L CNN
+F 4 "FDD7N25LZTM" H 5550 2450 60  0001 C CNN "MPN"
 	1    5550 2450
 	1    0    0    -1
@@
 P 5900 5800
 F 0 "Q3" H 6100 5875 50  0000 L CNN
-F 1 "FDD18N20LZ" H 6100 5800 50  0000 L CNN
+F 1 "FDD7N25LZTM" H 6100 5800 50  0000 L CNN
 F 2 "TO_SOT_Packages_SMD:TO-252-2Lead" H 6100 5725 50  0001 L CIN
-F 3 "https://www.digikey.com/product-detail/en/on-semiconductor/FDD18N20LZ/FDD18N20LZCT-ND/3908087" H 5900 5800 50  0001 L CNN
-F 4 "FDD18N20LZ" H 5900 5800 60  0001 C CNN "MPN"
+F 3 "https://www.digikey.com/product-detail/en/on-semiconductor/FDD7N25LZTM/FDD7N25LZTMCT-ND/3908038" H 5900 5800 50  0001 L CNN
+F 4 "FDD7N25LZTM" H 5900 5800 60  0001 C CNN "MPN"
 	1    5900 5800
 	1    0    0    -1

Commit message: adjusted the gate resistor for increased bandwidth
Parts:
- R2, R9: value 8.2k -> 1k
Changed lines of the file:
@@
 P 4950 2650
 F 0 "R2" V 5030 2650 50  0000 C CNN
-F 1 "8.2k" V 4950 2650 50  0000 C CNN
+F 1 "1k" V 4950 2650 50  0000 C CNN
 F 2 "Resistors_SMD:R_0805_HandSoldering" V 4880 2650 50  0001 C CNN
-F 3 "https://www.digikey.com/product-detail/en/yageo/RC0805FR-078K2L/311-8.20KCRCT-ND/731094" H 4950 2650 50  0001 C CNN
+F 3 "https://www.digikey.com/product-detail/en/yageo/RC0805FR-071KL/311-1.00KCRCT-ND/730391" H 4950 2650 50  0001 C CNN
 F 4 "RC0805FR-078K2L" V 4950 2650 60  0001 C CNN "MPN"
 	1    4950 2650
@@
 P 5300 6000
 F 0 "R9" V 5380 6000 50  0000 C CNN
-F 1 "8.2k" V 5300 6000 50  0000 C CNN
+F 1 "1k" V 5300 6000 50  0000 C CNN
 F 2 "Resistors_SMD:R_0805_HandSoldering" V 5230 6000 50  0001 C CNN
-F 3 "https://www.digikey.com/product-detail/en/yageo/RC0805FR-078K2L/311-8.20KCRCT-ND/731094" H 5300 6000 50  0001 C CNN
+F 3 "https://www.digikey.com/product-detail/en/yageo/RC0805FR-071KL/311-1.00KCRCT-ND/730391" H 5300 6000 50  0001 C CNN
 F 4 "RC0805FR-078K2L" V 5300 6000 60  0001 C CNN "MPN"
 	1    5300 6000
