File: KC_NixieBargraphHat/NixieBargraphHat.kicad_pcb (KiCad board)
At the start: 2 copper layers, 50 parts, among them J1 Screw_Terminal_1x03, J2 Screw_Terminal_1x02, J3 Screw_Terminal_1x03, J4 Screw_Terminal_1x03, Q1 FDD18N20LZ, Q2 2N7002, Q3 FDD18N20LZ, Q4 2N7002, U1 MCP6411, U2 Raspberry_PI_Zero_Header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

Commit message: added gerber files
Parts:
- moved R7 0.13 mm to (130.0, 111.3)
- moved R6 0.07 mm to (127.1, 111.4)
Other:
- board outline added: 65 x 30 mm
- rule pad_to_mask_clearance: 0.2 -> 0.0508

Commit message: Updated the follwoing changes: 1. Adjusted the gate resistor BOM to include a 1kohm resistor to gate of mosfet 2. updated silk screen to add labels for each of the Nixie tube and power supply connections.
Other:
- board text added: "+5v"
- board text added: "170v"
- board text added: "A"
- board text added: "Aux_C"
- board text added: "C"
- board text added: "EN"
- board text added: "GND"
Changed lines of the file:
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@@
     (area 103.314999 85.414999 168.475001 115.585001)
     (thickness 1.6)
-    (drawings 12)
+    (drawings 22)
     (tracks 565)
     (zones 0)
@@
     (pad_to_mask_clearance 0.0508)
     (aux_axis_origin 0 0)
-    (visible_elements FFFCFF7F)
+    (visible_elements FFFEFF7F)
     (pcbplotparams
       (layerselection 0x010f0_80000001)
@@
     (at 164.69 106.39 90)
     (descr "3-way 2.54mm pitch terminal block, Phoenix MPT series")
-    (fp_text reference J1 (at -2.69 -2.27 90) (layer F.SilkS)
+    (fp_text reference J1 (at -2.61 2.31 90) (layer F.SilkS)
       (effects (font (size 1 1) (thickness 0.15)))
     )
@@
       (effects (font (size 1 1) (thickness 0.15)))
     )
-    (fp_text user %R (at -2.69 -2.21 90) (layer F.Fab)
+    (fp_text user %R (at -2.61 2.41 90) (layer F.Fab)
       (effects (font (size 1 1) (thickness 0.15)))
     )
@@
     (at 164.69 97.49 90)
     (descr "2-way 2.54mm pitch terminal block, Phoenix MPT series")
-    (fp_text reference J2 (at 1.27 -4.50088 90) (layer F.SilkS)
+    (fp_text reference J2 (at 4.99 2.51 90) (layer F.SilkS)
       (effects (font (size 1 1) (thickness 0.15)))
     )
@@
       (effects (font (size 1 1) (thickness 0.15)))
     )
-    (fp_text user %R (at 1.15 -4.29 90) (layer F.Fab)
+    (fp_text user %R (at 5.09 2.41 90) (layer F.Fab)
       (effects (font (size 1 1) (thickness 0.15)))
     )
@@
     (tags "resistor 0805")
     (attr smd)
-    (fp_text reference R14 (at -3.83 0.11 180) (layer F.SilkS)
+    (fp_text reference R14 (at -3.68 0.66 180) (layer F.SilkS)
       (effects (font (size 1 1) (thickness 0.15)))
     )
@@
       (xy -1.51384 -2.24536)) (layer B.SilkS) (width 0.00254))
   )
+  (gr_text GND (at 160.9 100.6 90) (layer F.SilkS)
+    (effects (font (size 0.75 0.75) (thickness 0.1)))
+  )
+  (gr_text EN (at 160.3 104.2 90) (layer F.SilkS)
+    (effects (font (size 0.75 0.75) (thickness 0.1)))
+  )
+  (gr_text +5v (at 160.6 108.4 90) (layer F.SilkS)
+    (effects (font (size 0.75 0.75) (thickness 0.1)))
+  )
+  (gr_text Aux_C (at 118.4 114.2) (layer F.SilkS)
+    (effects (font (size 0.75 0.75) (thickness 0.1)))
+  )
+  (gr_text C (at 115.2 114.2) (layer F.SilkS)
+    (effects (font (size 0.75 0.75) (thickness 0.1)))
+  )
+  (gr_text A (at 112.5 114.3) (layer F.SilkS)
+    (effects (font (size 0.75 0.75) (thickness 0.1)))
+  )
+  (gr_text C (at 149.3 114.3) (layer F.SilkS)
+    (effects (font (size 0.75 0.75) (thickness 0.1)))
+  )
+  (gr_text Aux_C (at 152.1 114.4) (layer F.SilkS)
+    (effects (font (size 0.75 0.75) (thickness 0.1)))
+  )
+  (gr_text A (at 147 114.3) (layer F.SilkS)
+    (effects (font (size 0.75 0.75) (thickness 0.1)))
+  )
+  (gr_text 170v (at 160.9 95.7 90) (layer F.SilkS)
+    (effects (font (size 0.75 0.75) (thickness 0.1)))
+  )
   (dimension 30.03 (width 0.3) (layer F.Fab)

Commit message: Added all the changes for Part 2 of the Hat.   UPdated silksceen, reduced R2 and R9, new gerbers (Part 2). The original gerbers were saved.
Other:
- board text added: "NixieBarGraphHat Rev2_1939"
- board text removed: "NixieBarGraphHat Rev1_1906"
Changed lines of the file:
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@@
     (links 96)
     (no_connects 0)
-    (area 103.314999 85.414999 168.475001 115.585001)
+    (area 102.2951 77.39 180.88 116.414601)
     (thickness 1.6)
     (drawings 22)
@@
     (tags "resistor 0805")
     (attr smd)
-    (fp_text reference R5 (at 3.01 -0.15 360) (layer F.SilkS)
+    (fp_text reference R5 (at 3.13 -0.79 360) (layer F.SilkS)
       (effects (font (size 1 1) (thickness 0.15)))
     )
@@
     (tags "resistor 0805")
     (attr smd)
-    (fp_text reference R15 (at 3.13152 0.92592 360) (layer F.SilkS)
+    (fp_text reference R15 (at 3.01152 0.68592 360) (layer F.SilkS)
       (effects (font (size 1 1) (thickness 0.15)))
     )
@@
     (tags "resistor 0805")
     (attr smd)
-    (fp_text reference R16 (at 3.1001 -1.3019 360) (layer F.SilkS)
+    (fp_text reference R16 (at 3.0801 -0.5219 360) (layer F.SilkS)
       (effects (font (size 1 1) (thickness 0.15)))
     )
@@
     (tags "resistor 0805")
     (attr smd)
-    (fp_text reference R17 (at 3.0882 0.3034 360) (layer F.SilkS)
+    (fp_text reference R17 (at 3.1682 0.2634 360) (layer F.SilkS)
       (effects (font (size 1 1) (thickness 0.15)))
     )
@@
       (xy -1.51384 -2.24536)) (layer B.SilkS) (width 0.00254))
   )
-  (gr_text GND (at 160.9 100.6 90) (layer F.SilkS)
+  (gr_text GND (at 160.04 101.64 90) (layer F.SilkS)
     (effects (font (size 0.75 0.75) (thickness 0.1)))
   )
-  (gr_text EN (at 160.3 104.2 90) (layer F.SilkS)
+  (gr_text EN (at 159.92 104.34 90) (layer F.SilkS)
     (effects (font (size 0.75 0.75) (thickness 0.1)))
   )
-  (gr_text +5v (at 160.6 108.4 90) (layer F.SilkS)
+  (gr_text +5v (at 160 107.25 90) (layer F.SilkS)
     (effects (font (size 0.75 0.75) (thickness 0.1)))
   )
@@
     (effects (font (size 1 1) (thickness 0.2)) (justify mirror))
   )
-  (gr_text "NixieBarGraphHat Rev1_1906" (at 128.09 114.19) (layer B.SilkS)
+  (gr_text "NixieBarGraphHat Rev2_1939" (at 128.09 114.19) (layer B.SilkS)
     (effects (font (size 1.5 1.5) (thickness 0.3)) (justify mirror))
   )
